File: XBEE Grove C/XBEE SMD Pin Headers + Grove Drivers.kicad_sch (KiCad schematic)
At the start: 9 parts, among them J10 110990030, J11 110990030, J4 110990030, J5 110990030, J6 110990030, J7 110990030, J8 110990030, J9 110990030

Commit message: Add files via upload
Updated to v2 (all connectors now have the same number scheme as the original).
Parts:
- removed J1: ~, XBEE_Grove_C:XBEE_SMT, symbol XBEE_Grove_C:XBEE_SMT
- added FID1, FID2: Fiducial, Fiducial:Fiducial_1mm_Mask2mm, symbol Mechanical:Fiducial
- added J12: ~, XBEE_Grove_C:XBEE_SMT_P14-21, symbol XBEE_Grove_C:XBEE_SMT_P14-21
- added J13: ~, XBEE_Grove_C:XBEE_SMT_P22-34, symbol XBEE_Grove_C:XBEE_SMT_P22-34
- added J9: ~, XBEE_Grove_C:XBEE_SMT_P1-13, symbol XBEE_Grove_C:XBEE_SMT_P1-13
- renumbered J4 to J1, J10 to J14, J11 to J15, J5 to J2, J6 to J3, J7 to J4, J8 to J5, J9 to J6
Connections:
- net +3.3V: now also J13.27 (VREF), J9.2 (VCC)
- net AD0/CB: now also J13.33 (COMM/AD0/DIO0)
- net AD2: now also J13.31 (AD2/DIO2)
- net AD3: now also J13.30 (AD3/DIO3)
- net ASSOC_LED: now also J13.28 (ASSOC/DIO5)
- net DIO11/I2C_SDA: now also J9.8 (PWM1/DIO11)
- net DIO12: now also J9.5 (DIO12)
- net DIO18: now also J12.21 (SPI_SCLK/DIO18)
- net DIO19: now also J9.12 (ATTN/DIO19)
- net DIO1/I2C_SCL: now also J13.32 (AD1/DIO1)
- net DIO4: now also J13.24 (DIO4)
- net DIO9: now also J13.26 (ON/SLP/DIO9)
- net GND: now also J13.22 (GND), J9.1 (GND), J9.11 (GND), J9.13 (GND)
- net RESET_N: now also J9.6 (RESET)
- net RSSI/PWM0: now also J9.7 (PWM/RSSI//DIO10)
- net XBEE_CTS_N: now also J13.25 (CTS/DIO7)
- net XBEE_DTR_N: now also J9.10 (DTR/DIO8)
- net XBEE_RTS_N: now also J13.29 (RTS/DIO6)
- net XBEE_RX: now also J9.4 (DIN/CONFIG/DIO14)
- net XBEE_TX: now also J9.3 (DOUT/DIO13)

Commit message: Add files via upload
Included 76002056 part number for the SMT connectors.
Parts:
- J12, J13, J9: value ~ -> 76002056
